File: hardware/shen.kicad_pcb (KiCad board)
At the start: 2 copper layers, 21 x 51 mm, 48 parts, among them J1 Conn_01x20_Pin, J2 Conn_01x20_Pin, J3 Conn_01x03_Pin, J4 USB_C_Receptacle_USB2.0_16P, SW1 SW_Push, SW2 SW_Push, U1 RP2350A, U2 W25Q32JVZP, U3 RPI-RM2, U4 TLV62084DSGx, Y1 12MHz

Commit message: pcb work
Parts:
- removed C3: 4.7u, Capacitor_SMD:C_0603_1608Metric
- moved C19 78.1 mm to (182.0, 90.0), turned to 90 degrees
- moved L2 73.9 mm to (179.8, 92.5), turned to 180 degrees
- moved C20 72.4 mm to (181.1, 88.1)
- moved C17 71.8 mm to (177.3, 91.7), turned to 90 degrees
- moved C4 68.5 mm to (178.5, 98.1)
- moved C2 68.0 mm to (178.4, 94.2)
- moved C1 68.0 mm to (181.4, 99.2), turned to -90 degrees
- moved C8 65.3 mm to (180.2, 100.0), turned to 90 degrees
- moved L1 64.2 mm to (178.4, 96.1)
- moved C13 63.8 mm to (178.4, 90.9), turned to 90 degrees
- moved C5 63.5 mm to (181.2, 102.8)
- moved R10 63.0 mm to (179.4, 88.0)
- moved R4 61.5 mm to (180.2, 98.3), turned to 90 degrees
- moved C7 61.1 mm to (175.5, 98.0), turned to 90 degrees
- moved R9 60.5 mm to (178.4, 89.2), turned to 90 degrees
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Routing:
- net +3V3: track 0.00 -> 54.4 mm, vias 0 -> 10
- net GND: track 0.00 -> 29.8 mm, vias 2 -> 30
- net /GP16: track 0.00 -> 28.5 mm, vias 0 -> 1
- net /GP29: track 0.00 -> 28.3 mm, vias 0 -> 2
- net /GP15: track 0.00 -> 27.2 mm, vias 0 -> 1
- net /GP17: track 0.00 -> 26.9 mm, vias 0 -> 1
- net /GP24: track 0.00 -> 26.5 mm, vias 0 -> 4
- net +1V1: track 0.00 -> 26.0 mm
- net /GP14: track 0.00 -> 24.0 mm, vias 0 -> 1
- net /GP0: track 0.00 -> 22.7 mm, vias 0 -> 1
- net /GP1: track 0.00 -> 20.7 mm, vias 0 -> 1
- net /GP23: track 0.00 -> 19.6 mm, vias 0 -> 2
- net /GP25: track 0.00 -> 18.3 mm, vias 0 -> 2
- net /GP13: track 0.00 -> 17.9 mm
- net /GP18: track 0.00 -> 17.8 mm
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- added copper zone on B.Cu, net GND
- added copper zone on F.Cu, net GND

Commit message: PCB complete
Parts:
- moved R11 0.67 mm to (181.5, 117.8)
- moved C20 0.38 mm to (181.5, 88.0)
- moved R8 0.27 mm to (171.1, 97.9)
- moved U3 0.17 mm to (175.6, 126.8)
- moved C14 0.15 mm to (169.7, 117.7)
- moved C19 0.13 mm to (182.0, 90.1)
- moved R4 0.08 mm to (180.3, 98.3)
- moved R6 0.07 mm to (169.2, 91.0)
Connections:
- J1 pad 10: unconnected-(J1-Pin_10-Pad10) -> +3V3
- J1 pad 4: unconnected-(J1-Pin_4-Pad4) -> GND
Routing:
- net +3V3: track 54.4 -> 31.2 mm, vias 10 -> 16
- net /RUN: track 5.91 -> 14.7 mm, vias 0 -> 1
- net VBUS: track 2.19 -> 4.57 mm, vias 0 -> 4
- net Net-(U4-SW): track 0.00 -> 1.70 mm
- net +1V1: track 26.0 -> 24.9 mm
- net /GP24: track 26.5 -> 25.4 mm
- net Net-(U4-FB): track 1.07 -> 1.81 mm
- net /GP23: track 19.6 -> 18.8 mm
- net /XIN: track 7.43 -> 8.13 mm
- net /GP15: track 27.2 -> 26.5 mm
- net /GP16: track 28.5 -> 27.9 mm
- net /GP0: track 22.7 -> 22.1 mm
- net /USB_DN: track 7.63 -> 8.19 mm
- net /GP17: track 26.9 -> 26.3 mm
- net /GP13: track 17.9 -> 17.4 mm
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- added copper zone on F.Cu, net +3V3
- added copper zone on In2.Cu, net +3V3
- added copper zone on In1.Cu, net GND
- added copper zone on F.Cu, net VBUS
- added copper zone on In2.Cu, net VBUS
Other:
- copper layers 2 -> 4
